Commit message: Incorporate Review Commments

File: Project_2_Robochase/my_robot/urdf/my_robot.xacro (robot description, xacro)
@@ -2,4 +2,16 @@
 <robot name="my_robot" xmlns:xacro="http://www.ros.org/wiki/xacro">
   <xacro:include filename="$(find my_robot)/urdf/my_robot.gazebo" />
+  <gazebo reference="left_wheel">
+    <material>Gazebo/Blue</material>
+  </gazebo>
+  <gazebo reference="right_wheel">
+    <material>Gazebo/Blue</material>
+  </gazebo>
+  <gazebo reference="camera">
+    <material>Gazebo/Red</material>
+  </gazebo>
+  <gazebo reference="chassis">
+    <material>Gazebo/Yellow</material>
+  </gazebo>
   <link name="robot_footprint"></link>
   <joint name="robot_footprint_joint" type="fixed">
@@ -8,20 +20,71 @@
     <child link="chassis" />
   </joint>
+  <joint name="camera_joint" type="fixed">
+    <origin xyz="0.2 0 0" rpy="0 0 0" />
+    <parent link="chassis"/>
+    <child link="camera" />
+    <axis xyz="0 1 0"/>
+  </joint>
   <joint name="hokuyo_joint" type="fixed">
-    <origin xyz="0.35 0 0.1" rpy="0 0 0" />
+    <origin xyz="0.15 0 0.1" rpy="0 0 0" />
     <parent link="chassis"/>
     <child link="hokuyo" />
-    <axis xyz="0 1 0" rpy="0 0 0"/>
+    <axis xyz="0 1 0"/>
   </joint>
-  <link name='hokuyo'>
+  <joint type="continuous" name="left_wheel_hinge">
+    <origin xyz="0 0.23 0" rpy="0 0 0" />
+    <parent link="chassis"/>
+    <child link="left_wheel" />
+    <axis xyz="0 1 0" rpy="0 0 0" />
+    <limit effort="10000" velocity="1000" />
+    <dynamics damping="1.0" friction="1.0" />
+  </joint>
+  <joint type="continuous" name="right_wheel_hinge">
+    <origin xyz="0 -0.23 0" rpy="0 0 0" />
+    <parent link="chassis"/>
+    <child link="right_wheel" />
+    <axis xyz="0 1 0" rpy="0 0 0" />
+    <limit effort="10000" velocity="1000" />
+    <dynamics damping="1.0" friction="1.0" />
+  </joint>
+  <link name="camera">
     <inertial>
-    <origin xyz="0 0 0" rpy="0 0 0"/>
-    <mass value="1e-5"/>
+      <mass value="0.1"/>
+      <origin xyz="0 0 0" rpy="0 0 0"/>
       <inertia
-          ixx="1e-6" ixy="0" ixz="0"
-          iyy="1e-6" iyz="0"
-          izz="1e-6"
+        ixx="1e-6" ixy="0.0" ixz="0.0"
+        iyy="1e-6" iyz="0.0"
+        izz="1e-6"
       />
     </inertial>
+    <collision>
+      <origin xyz="0 0 0" rpy="0 0 0"/>
+      <geometry>
+        <box size="0.05 0.05 0.05"/>
+      </geometry>
+    </collision>
+    <visual>
+      <origin xyz="0 0 0" rpy="0 0 0"/>
+      <geometry>
+        <box size="0.05 0.05 0.05"/>
+      </geometry>
+    </visual>
+  </link>
+  <link name="hokuyo">
+    <inertial>
+      <mass value="1e-5"/>
+      <origin xyz="0 0 0" rpy="0 0 0"/>
+      <inertia
+        ixx="1e-6" ixy="0.0" ixz="0.0"
+        iyy="1e-6" iyz="0.0"
+        izz="1e-6"
+      />
+    </inertial>
+    <collision>
+      <origin xyz="0 0 0" rpy="0 0 0"/>
+      <geometry>
+        <box size="0.1 0.1 0.1"/>
+      </geometry>
+    </collision>
     <visual>
       <origin xyz="0 0 0" rpy="0 0 0"/>
@@ -30,101 +93,50 @@
       </geometry>
     </visual>
+  </link>
+  <link name="left_wheel">
+    <inertial>
+      <mass value="5"/>
+      <origin xyz="0 0 0" rpy="0 1.5707 1.5707"/>
+      <inertia
+        ixx="0.1" ixy="0.0" ixz="0.0"
+        iyy="0.1" iyz="0.0"
+        izz="0.1"
+      />
+    </inertial>
     <collision>
-      <origin xyz="0 0 0" rpy="0 0 0"/>
+      <origin xyz="0 0 0" rpy="0 1.5707 1.5707"/>
       <geometry>
-        <box size="0.1 0.1 0.1"/>
+        <cylinder radius="0.1" length="0.2"/>
       </geometry>
     </collision>
-  </link>
-  <joint name="camera_joint" type="fixed">
-    <origin xyz="0.4 0 0" rpy="0 0 0" />
-    <parent link="chassis"/>
-    <child link="camera" />
-    <axis xyz="0 1 0" rpy="0 0 0"/>
-  </joint>
-  <link name='camera'>
-    <inertial>
-    <origin xyz="0 0 0" rpy="0 0 0"/>
-    <mass value="0.1"/>
-      <inertia
-          ixx="1e-6" ixy="0" ixz="0"
-          iyy="1e-6" iyz="0"
-          izz="1e-6"
-      />
-    </inertial>
-    <visual>
-      <origin xyz="0 0 0" rpy="0 0 0"/>
-      <geometry>
-        <box size="0.05 0.05 0.05"/>
-      </geometry>
-    </visual>
-    <collision>
-      <origin xyz="0 0 0" rpy="0 0 0"/>
-      <geometry>
-        <box size="0.05 0.05 0.05"/>
-      </geometry>
-    </collision>
-  </link>
-  <joint name="left_wheel_hinge" type="continuous">
-    <origin xyz="0 0.15 0" rpy="0 0 0" />
-    <parent link="chassis"/>
-    <child link="left_wheel" />
-    <axis xyz="0 1 0" rpy="0 0 0"/>
-    <limit effort="10000" velocity="1000"/>
-    <dynamics damping="1.0" friction="1.0"/>
-  </joint>
-  <joint name="right_wheel_hinge" type="continuous">
-    <origin xyz="0 0.15 0" rpy="0 0 0" />
-    <parent link="chassis"/>
-    <child link="right_wheel" />
-    <axis xyz="0 1 0" rpy="0 0 0"/>
-    <limit effort="10000" velocity="1000"/>
-    <dynamics damping="1.0" friction="1.0"/>
-  </joint>
-  <link name='left_wheel'>
-    <inertial>
-    <origin xyz="0 0 0" rpy="0 1.5707 1.5707"/>
-    <mass value="5"/>
-      <inertia
-          ixx="0.1" ixy="0" ixz="0"
-          iyy="0.1" iyz="0"
-          izz="0.1"
-      />
-    </inertial>
     <visual>
       <origin xyz="0 0 0" rpy="0 1.5707 1.5707"/>
       <geometry>
-        <cylinder radius="0.1" length="0.05"/>
+        <cylinder radius="0.1" length="0.2"/>
       </geometry>
     </visual>
+  </link>
+  <link name="right_wheel">
+    <inertial>
+      <mass value="5"/>
+      <origin xyz="0 0 0" rpy="0 1.5707 1.5707"/>
+      <inertia
+        ixx="0.1" ixy="0.0" ixz="0.0"
+        iyy="0.1" iyz="0.0"
+        izz="0.1"
+      />
+    </inertial>
     <collision>
       <origin xyz="0 0 0" rpy="0 1.5707 1.5707"/>
       <geometry>
-        <cylinder radius="0.1" length="0.05"/>
+        <cylinder radius="0.1" length="0.2"/>
       </geometry>
     </collision>
-  </link>
-  <link name='right_wheel'>
-    <inertial>
-    <origin xyz="0 -0.3 0" rpy="0 1.5707 1.5707"/>
-    <mass value="5"/>
-      <inertia
-          ixx="0.1" ixy="0" ixz="0"
-          iyy="0.1" iyz="0"
-          izz="0.1"
-      />
-    </inertial>
     <visual>
-      <origin xyz="0 -0.3 0" rpy="0 1.5707 1.5707"/>
+      <origin xyz="0 0 0" rpy="0 1.5707 1.5707"/>
       <geometry>
-        <cylinder radius="0.1" length="0.05"/>
+        <cylinder radius="0.1" length="0.2"/>
       </geometry>
     </visual>
-    <collision>
-      <origin xyz="0 -0.3 0" rpy="0 1.5707 1.5707"/>
-      <geometry>
-        <cylinder radius="0.1" length="0.05"/>
-      </geometry>
-    </collision>
   </link>
   <link name='chassis'>
@@ -148,9 +160,9 @@
       <origin xyz="0 0 0" rpy=" 0 0 0"/>
       <geometry>
-        <box size=".8 .2 .1"/>
+        <box size=".4 .2 .1"/>
       </geometry>
     </visual>
     <collision name='back_caster_collision'>
-      <origin xyz="-0.35 0 -0.05" rpy=" 0 0 0"/>
+      <origin xyz="-0.15 0 -0.05" rpy=" 0 0 0"/>
       <geometry>
         <sphere radius="0.0499"/>
@@ -158,5 +170,5 @@
     </collision>
     <visual name='back_caster_visual'>
-      <origin xyz="-0.35 0 -0.05" rpy=" 0 0 0"/>
+      <origin xyz="-0.15 0 -0.05" rpy=" 0 0 0"/>
       <geometry>
         <sphere radius="0.05"/>
@@ -164,5 +176,5 @@
     </visual>
     <collision name='front_caster_collision'>
-      <origin xyz="0.35 0 -0.05" rpy=" 0 0 0"/>
+      <origin xyz="0.15 0 -0.05" rpy=" 0 0 0"/>
       <geometry>
         <sphere radius="0.0499"/>
@@ -170,5 +182,5 @@
     </collision>
     <visual name='front_caster_visual'>
-      <origin xyz="0.35 0 -0.05" rpy=" 0 0 0"/>
+      <origin xyz="0.15 0 -0.05" rpy=" 0 0 0"/>
       <geometry>
         <sphere radius="0.05"/>
@@ -176,15 +188,3 @@
     </visual>
   </link>
-  <gazebo reference="chassis">
-    <material>Gazebo/Green</material>
-  </gazebo>
-  <gazebo reference="left_wheel">
-    <material>Gazebo/Yellow</material>
-  </gazebo>
-  <gazebo reference="right_wheel">
-    <material>Gazebo/Yellow</material>
-  </gazebo>
-  <gazebo reference="camera">
-    <material>Gazebo/Blue</material>
-  </gazebo>
 </robot>
